Commit message: new update

File: URDF/Spyder_it_doesnt_walk/spider_description.urdf (robot description, URDF)
Before this commit: robot spider_robot, 13 links, 12 joints
Links:
- link FL_calf_link: mass 0.02 -> 0.055
- link FL_hip_link: mass 0.05 -> 0.055
- link FL_thigh_link: mass 0.03 -> 0.055
- link FR_calf_link: mass 0.02 -> 0.055
- link FR_hip_link: mass 0.05 -> 0.055
- link FR_thigh_link: mass 0.03 -> 0.055
- link RL_calf_link: mass 0.02 -> 0.055
- link RL_hip_link: mass 0.05 -> 0.055
- link RL_thigh_link: mass 0.03 -> 0.055
- link RR_calf_link: mass 0.02 -> 0.055
- link RR_hip_link: mass 0.05 -> 0.055
- link RR_thigh_link: mass 0.03 -> 0.055
- link base_link: mass 0.5 -> 0.05
Joints:
- joint FL_calf_joint: limit lower=-0.3 upper=1.57 effort=20 velocity=1.57 -> lower=-0.3 upper=1.57 effort=1
- joint FL_hip_joint: limit lower=-0.785 upper=0.785 effort=20 velocity=1.57 -> lower=-0.785 upper=0.785 effort=1
- joint FL_thigh_joint: limit lower=-0.9 upper=0.9 effort=20 velocity=1.57 -> lower=-0.9 upper=0.9 effort=1
- joint FR_calf_joint: limit lower=-0.3 upper=1.57 effort=20 velocity=1.57 -> lower=-0.3 upper=1.57 effort=1
- joint FR_hip_joint: limit lower=-0.785 upper=0.785 effort=20 velocity=1.57 -> lower=-0.785 upper=0.785 effort=1
- joint FR_thigh_joint: limit lower=-0.9 upper=0.9 effort=20 velocity=1.57 -> lower=-0.9 upper=0.9 effort=1
- joint RL_calf_joint: limit lower=-0.3 upper=1.57 effort=20 velocity=1.57 -> lower=-0.3 upper=1.57 effort=1
- joint RL_hip_joint: limit lower=-0.785 upper=0.785 effort=20 velocity=1.57 -> lower=-0.785 upper=0.785 effort=1
- joint RL_thigh_joint: limit lower=-0.9 upper=0.9 effort=20 velocity=1.57 -> lower=-0.9 upper=0.9 effort=1
- joint RR_calf_joint: limit lower=-0.3 upper=1.57 effort=20 velocity=1.57 -> lower=-0.3 upper=1.57 effort=1
- joint RR_hip_joint: limit lower=-0.785 upper=0.785 effort=20 velocity=1.57 -> lower=-0.785 upper=0.785 effort=1
- joint RR_thigh_joint: limit lower=-0.9 upper=0.9 effort=20 velocity=1.57 -> lower=-0.9 upper=0.9 effort=1
