Commit message: updated urdf big_bertha with ydlidar X2

File: assets/URDF/Spyder_mg995_description.urdf (robot description, URDF)
Before this commit: robot SpdrBot, 13 links, 12 joints
Links:
- added link lidar_link, mass 0.055231; collision mesh filename=./meshes/ydlidar.stl scale=0.0001 0.0001 0.0001; visual mesh filename=./meshes/ydlidar.stl scale=0.0001 0.0001 0.0001
Joints:
- added joint lidar joint: type fixed, parent base_link, child lidar_link, origin xyz=0.01 0 0 rpy=0 0 0, axis 0 0 0

Commit message: fix/issue #21 #22 #23 addressed

File: assets/URDF/Spyder_mg995_description.urdf (robot description, URDF)
Before this commit: robot SpdrBot, 14 links, 13 joints
Links:
- link arm_a_1_1: mass 0.5428876729051647 -> 0.12
- link arm_a_2_1: mass 0.5428876729051773 -> 0.12
- link arm_a_3_1: mass 0.5428876729051227 -> 0.12
- link arm_a_4_1: mass 0.5428876729051186 -> 0.12
- link arm_b_1_1: mass 0.34922835365489313 -> 0.10
- link arm_b_2_1: mass 0.3492283536549301 -> 0.10
- link arm_b_3_1: mass 0.34922833079669513 -> 0.10; geometry collision mesh filename=./meshes/arm_b_3_1.stl scale=0.001 0.001 0.001; visual mesh filename=./meshes/arm_b_3_1.stl scale=0.001 0.001 0.001
- link arm_b_4_1: mass 0.3492283307966938 -> 0.10
- link arm_c_1_1: mass 0.8577978208262385 -> 0.12
- link arm_c_2_1: mass 0.8577978208264597 -> 0.12
- link arm_c_3_1: mass 0.8577978208264664 -> 0.12
- link arm_c_4_1: mass 0.8577978208262359 -> 0.12
- link base_link: mass 2.886187908245162 -> 0.35
- link lidar_link: mass 0.055231 -> 0.126; geometry visual mesh filename=./meshes/ydlidar.stl scale=0.0001 0.0001 0.0001
Joints:
- removed joint Revolute 110
- removed joint Revolute 111
- removed joint Revolute 112
- removed joint Revolute 114
- removed joint Revolute 115
- removed joint Revolute 116
- removed joint Revolute 117
- removed joint Revolute 118
- removed joint Revolute 119
- removed joint Revolute 120
- removed joint Revolute 121
- removed joint lidar joint
- added joint Revolute_110: type continuous, parent base_link, child arm_a_4_1, origin xyz=-0.0802 -0.0649 0.0278 rpy=0 0 0, axis 0.0 -0.0 1.0
- added joint Revolute_111: type continuous, parent arm_a_4_1, child arm_b_4_1, origin xyz=-0.015981 -0.055296 -0.0141 rpy=0 0 0, axis 0.707107 -0.707107 0.0
- added joint Revolute_112: type continuous, parent arm_b_4_1, child arm_c_4_1, origin xyz=-0.028284 -0.028284 0.069282 rpy=0 0 0, axis -0.707107 0.707107 -0.0
- added joint Revolute_114: type continuous, parent arm_a_1_1, child arm_b_1_1, origin xyz=0.055296 -0.015981 -0.0141 rpy=0 0 0, axis 0.707107 0.707107 0.0
- added joint Revolute_115: type continuous, parent arm_b_1_1, child arm_c_1_1, origin xyz=0.028284 -0.028284 0.069282 rpy=0 0 0, axis -0.707107 -0.707107 -0.0
- added joint Revolute_116: type continuous, parent base_link, child arm_a_2_1, origin xyz=0.0802 0.0649 0.0278 rpy=0 0 0, axis -0.0 0.0 1.0
- added joint Revolute_117: type continuous, parent arm_a_2_1, child arm_b_2_1, origin xyz=0.015981 0.055296 -0.0141 rpy=0 0 0, axis -0.707107 0.707107 -0.0
- added joint Revolute_118: type continuous, parent arm_b_2_1, child arm_c_2_1, origin xyz=0.028284 0.028284 0.069282 rpy=0 0 0, axis 0.707107 -0.707107 -0.0
- added joint Revolute_119: type continuous, parent base_link, child arm_a_3_1, origin xyz=-0.0802 0.0649 0.0278 rpy=0 0 0, axis -0.0 0.0 1.0
- added joint Revolute_120: type continuous, parent arm_a_3_1, child arm_b_3_1, origin xyz=-0.055296 0.015981 -0.0141 rpy=0 0 0, axis -0.707107 -0.707107 0.0
- added joint Revolute_121: type continuous, parent arm_b_3_1, child arm_c_3_1, origin xyz=-0.028284 0.028284 0.069282 rpy=0 0 0, axis 0.707107 0.707107 -0.0
- added joint lidar_joint: type fixed, parent base_link, child lidar_link, origin xyz=0.01 0 0 rpy=0 0 0, axis 0 0 0
