Commit message: fix:urdf modified to have 3s2p type battery pack

File: assets/URDF/big_bertha/Spyder_mg995_description.urdf (robot description, URDF)
Before this commit: robot SpdrBot, 14 links, 13 joints
Links:
- added link battery_link, mass 0.2244; visual mesh filename=./meshes/battery_3s2p.stl scale=0.001 0.001 0.001
Joints:
- removed joint Revolute 113
- added joint Revolute_113: type continuous, parent base_link, child arm_a_1_1, origin xyz=0.0802 -0.0649 0.0278 rpy=0 0 0, axis 0.0 -0.0 1.0
- added joint battery_joint: type fixed, parent base_link, child battery_link, origin xyz=-0.04450 0.015 0.0065 rpy=0 0 0, axis 0 0 0
- joint lidar_joint: origin xyz=0.01 0 0 rpy=0 0 0 -> xyz=0.01 0.01 0.041 rpy=0 0 0

Commit message: feat: new urdf for big bertha is used

File: assets/URDF/big_bertha/Spyder_mg995_description.urdf (robot description, URDF)
Before this commit: robot SpdrBot, 15 links, 14 joints
Links:
- removed link lidar_link
- added link circuit_box_base_link, mass 0.016044; collision box size=0.102 0.1333 0.001; visual box size=0.102 0.1333 0.001
- added link circuit_box_link, mass 0.139015; collision box size=0.102 0.1333 0.001; collision mesh filename=./meshes/260519_PART_Body standoffs.STL scale=0.001 0.001 0.001
- added link ydlidar_link, mass 0.126000; collision mesh filename=./meshes/ydlidar.stl scale=0.0001 0.0001 0.0001; visual mesh filename=./meshes/ydlidar.stl scale=0.0001 0.0001 0.0001
- link arm_a_1_1: mass 0.12 -> 0.061703; geometry collision mesh filename=./meshes/260519_PART_Arm A Right.STL scale=0.001 0.001 0.001; collision mesh filename=./meshes/Servo_MG995.stl scale=0.001 0.001 0.001
- link arm_a_2_1: mass 0.12 -> 0.061703; geometry collision mesh filename=./meshes/260519_PART_Arm A Left.STL scale=0.001 0.001 0.001; collision mesh filename=./meshes/Servo_MG995.stl scale=0.001 0.001 0.001
- link arm_a_3_1: mass 0.12 -> 0.061703; geometry collision mesh filename=./meshes/260519_PART_Arm A Left.STL scale=0.001 0.001 0.001; collision mesh filename=./meshes/Servo_MG995.stl scale=0.001 0.001 0.001
- link arm_a_4_1: mass 0.12 -> 0.061703; geometry collision mesh filename=./meshes/260519_PART_Arm A Right.STL scale=0.001 0.001 0.001; collision mesh filename=./meshes/Servo_MG995.stl scale=0.001 0.001 0.001
- link arm_b_1_1: mass 0.10 -> 0.008137; geometry collision mesh filename=./meshes/260519_PART_Arm B.STL scale=0.001 0.001 0.001; visual mesh filename=./meshes/260519_PART_Arm B.STL scale=0.001 0.001 0.001
- link arm_b_2_1: mass 0.10 -> 0.008137; geometry collision mesh filename=./meshes/260519_PART_Arm B.STL scale=0.001 0.001 0.001; visual mesh filename=./meshes/260519_PART_Arm B.STL scale=0.001 0.001 0.001
- link arm_b_3_1: mass 0.10 -> 0.008137; geometry collision mesh filename=./meshes/260519_PART_Arm B.STL scale=0.001 0.001 0.001; visual mesh filename=./meshes/260519_PART_Arm B.STL scale=0.001 0.001 0.001
- link arm_b_4_1: mass 0.10 -> 0.008137; geometry collision mesh filename=./meshes/260519_PART_Arm B.STL scale=0.001 0.001 0.001; visual mesh filename=./meshes/260519_PART_Arm B.STL scale=0.001 0.001 0.001
- link arm_c_1_1: mass 0.12 -> 0.063683; geometry collision mesh filename=./meshes/260519_PART_Arm C Right.STL scale=0.001 0.001 0.001; collision mesh filename=./meshes/Servo_MG995.stl scale=0.001 0.001 0.001
- link arm_c_2_1: mass 0.12 -> 0.063683; geometry collision mesh filename=./meshes/260519_PART_Arm C Left.STL scale=0.001 0.001 0.001; collision mesh filename=./meshes/Servo_MG995.stl scale=0.001 0.001 0.001
- link arm_c_3_1: mass 0.12 -> 0.063683; geometry collision mesh filename=./meshes/260519_PART_Arm C Left.STL scale=0.001 0.001 0.001; collision mesh filename=./meshes/Servo_MG995.stl scale=0.001 0.001 0.001
- link arm_c_4_1: mass 0.12 -> 0.063683; geometry collision mesh filename=./meshes/260519_PART_Arm C Right.STL scale=0.001 0.001 0.001; collision mesh filename=./meshes/Servo_MG995.stl scale=0.001 0.001 0.001
- link base_link: mass 0.35 -> 0.263885; geometry collision mesh filename=./meshes/260519_PART_Arm perforated plate bottom.STL scale=0.001 0.001 0.001; collision mesh filename=./meshes/260519_PART_Arm perforated plate bottom.STL scale=0.001 0.001 0.001
- link battery_link: mass 0.2244 -> 0.500000; geometry collision box size=0.1083 0.07745 0.047; visual box size=0.1083 0.07745 0.047
Joints:
- removed joint lidar_joint
- added joint circuit_box_base_joint: type fixed, parent battery_link, child circuit_box_base_link, origin xyz=0 0 -0.0245 rpy=0 3.14 0
- added joint circuit_box_joint: type fixed, parent circuit_box_base_link, child circuit_box_link, origin xyz=0 0 0 rpy=0 0 0
- added joint ydlidar_joint: type fixed, parent circuit_box_link, child ydlidar_link, origin xyz=0 0 0 rpy=0 0 0
- joint Revolute_110: axis 0.0 -0.0 1.0 -> 0 1.0 0; limit (none) -> lower=-1.57 upper=1.57 effort=1.18 velocity=5.5; origin xyz=-0.0802 -0.0649 0.0278 rpy=0 0 0 -> xyz=0.129 0.02 -0.015 rpy=0 -0.785 0; type continuous -> revolute
- joint Revolute_111: axis 0.707107 -0.707107 0.0 -> 0 1.0 0; limit (none) -> lower=-1.57 upper=0.96 effort=1.18 velocity=5.5; origin xyz=-0.015981 -0.055296 -0.0141 rpy=0 0 0 -> xyz=0 -0.008 -0.052 rpy=0 1.57 1.57; type continuous -> revolute
- joint Revolute_112: axis -0.707107 0.707107 -0.0 -> 0 0 1; limit (none) -> lower=0 upper=2.355 effort=1.18 velocity=5.5; origin xyz=-0.028284 -0.028284 0.069282 rpy=0 0 0 -> xyz=0.08 0.03 0 rpy=0 1.57 1.57; type continuous -> revolute
- joint Revolute_113: axis 0.0 -0.0 1.0 -> 0 1.0 0; limit (none) -> lower=-1.57 upper=1.57 effort=1.18 velocity=5.5; origin xyz=0.0802 -0.0649 0.0278 rpy=0 0 0 -> xyz=-0.015 0.02 0.002 rpy=0 0.785 0; type continuous -> revolute
- joint Revolute_114: axis 0.707107 0.707107 0.0 -> 0 1.0 0; limit (none) -> lower=-1.57 upper=0.96 effort=1.18 velocity=5.5; origin xyz=0.055296 -0.015981 -0.0141 rpy=0 0 0 -> xyz=0 -0.008 -0.052 rpy=0 1.57 1.57; type continuous -> revolute
- joint Revolute_115: axis -0.707107 -0.707107 -0.0 -> 0 0 1; limit (none) -> lower=0 upper=2.355 effort=1.18 velocity=5.5; origin xyz=0.028284 -0.028284 0.069282 rpy=0 0 0 -> xyz=0.08 0.03 0 rpy=0 1.57 1.57; type continuous -> revolute
- joint Revolute_116: axis -0.0 0.0 1.0 -> 0 1.0 0; limit (none) -> lower=-1.57 upper=1.57 effort=1.18 velocity=5.5; origin xyz=0.0802 0.0649 0.0278 rpy=0 0 0 -> xyz=0.0027 0.02 0.145 rpy=0 2.355 0; type continuous -> revolute
- joint Revolute_117: axis -0.707107 0.707107 -0.0 -> 0 1.0 0; limit (none) -> lower=-1.57 upper=0.96 effort=1.18 velocity=5.5; origin xyz=0.015981 0.055296 -0.0141 rpy=0 0 0 -> xyz=0 -0.008 -0.052 rpy=0 1.57 1.57; type continuous -> revolute
- joint Revolute_118: axis 0.707107 -0.707107 -0.0 -> 0 0 1; limit (none) -> lower=0 upper=2.355 effort=1.18 velocity=5.5; origin xyz=0.028284 0.028284 0.069282 rpy=0 0 0 -> xyz=0.08 0.03 0 rpy=0 1.57 1.57; type continuous -> revolute
- joint Revolute_119: axis -0.0 0.0 1.0 -> 0 1.0 0; limit (none) -> lower=-1.57 upper=1.57 effort=1.18 velocity=5.5; origin xyz=-0.0802 0.0649 0.0278 rpy=0 0 0 -> xyz=0.145 0.02 0.128 rpy=0 -2.355 0; type continuous -> revolute
- joint Revolute_120: axis -0.707107 -0.707107 0.0 -> 0 1.0 0; limit (none) -> lower=-1.57 upper=0.96 effort=1.18 velocity=5.5; origin xyz=-0.055296 0.015981 -0.0141 rpy=0 0 0 -> xyz=0 -0.008 -0.052 rpy=0 1.57 1.57; type continuous -> revolute
- joint Revolute_121: axis 0.707107 0.707107 -0.0 -> 0 0 1; limit (none) -> lower=0 upper=2.355 effort=1.18 velocity=5.5; origin xyz=-0.028284 0.028284 0.069282 rpy=0 0 0 -> xyz=0.0775 0.03 0.001 rpy=0 1.57 1.57; type continuous -> revolute
- joint battery_joint: axis 0 0 0 -> (none); origin xyz=-0.04450 0.015 0.0065 rpy=0 0 0 -> xyz=0.0657 0.0385 0.0657 rpy=1.57 0 0

Commit message: feat: new urdf introduced

File: assets/URDF/big_bertha/Spyder_mg995_description.urdf (robot description, URDF)
Before this commit: robot SpdrBot, 17 links, 16 joints
Links:
- link arm_a_1_1: geometry collision mesh filename=./meshes/Servo_MG995.stl scale=0.001 0.001 0.001; collision mesh filename=./meshes/p_260519_PART_Arm_A_Right.STL scale=0.001 0.001 0.001
- link arm_a_2_1: geometry collision mesh filename=./meshes/Servo_MG995.stl scale=0.001 0.001 0.001; collision mesh filename=./meshes/p_260519_PART_Arm_A_Left.STL scale=0.001 0.001 0.001
- link arm_a_3_1: geometry collision mesh filename=./meshes/Servo_MG995.stl scale=0.001 0.001 0.001; collision mesh filename=./meshes/p_260519_PART_Arm_A_Left.STL scale=0.001 0.001 0.001
- link arm_a_4_1: geometry collision mesh filename=./meshes/Servo_MG995.stl scale=0.001 0.001 0.001; collision mesh filename=./meshes/p_260519_PART_Arm_A_Right.STL scale=0.001 0.001 0.001
- link arm_b_1_1: geometry collision mesh filename=./meshes/p_260519_PART_Arm_B.STL scale=0.001 0.001 0.001; visual mesh filename=./meshes/p_260519_PART_Arm_B.STL scale=0.001 0.001 0.001
- link arm_b_2_1: geometry collision mesh filename=./meshes/p_260519_PART_Arm_B.STL scale=0.001 0.001 0.001; visual mesh filename=./meshes/p_260519_PART_Arm_B.STL scale=0.001 0.001 0.001
- link arm_b_3_1: geometry collision mesh filename=./meshes/p_260519_PART_Arm_B.STL scale=0.001 0.001 0.001; visual mesh filename=./meshes/p_260519_PART_Arm_B.STL scale=0.001 0.001 0.001
- link arm_b_4_1: geometry collision mesh filename=./meshes/p_260519_PART_Arm_B.STL scale=0.001 0.001 0.001; visual mesh filename=./meshes/p_260519_PART_Arm_B.STL scale=0.001 0.001 0.001
- link arm_c_1_1: geometry collision mesh filename=./meshes/Servo_MG995.stl scale=0.001 0.001 0.001; collision mesh filename=./meshes/p_260519_PART_Arm_C_Right.STL scale=0.001 0.001 0.001
- link arm_c_2_1: geometry collision mesh filename=./meshes/Servo_MG995.stl scale=0.001 0.001 0.001; collision mesh filename=./meshes/p_260519_PART_Arm_C_Left.STL scale=0.001 0.001 0.001
- link arm_c_3_1: geometry collision mesh filename=./meshes/Servo_MG995.stl scale=0.001 0.001 0.001; collision mesh filename=./meshes/p_260519_PART_Arm_C_Left.STL scale=0.001 0.001 0.001
- link arm_c_4_1: geometry collision mesh filename=./meshes/Servo_MG995.stl scale=0.001 0.001 0.001; collision mesh filename=./meshes/p_260519_PART_Arm_C_Right.STL scale=0.001 0.001 0.001
- link base_link: geometry collision mesh filename=./meshes/Servo_MG995.stl scale=0.001 0.001 0.001; collision mesh filename=./meshes/Servo_MG995.stl scale=0.001 0.001 0.001
- link circuit_box_link: geometry collision box size=0.102 0.1333 0.001; collision mesh filename=./meshes/HW_688_LAYOUT.stl scale=0.001 0.001 0.001

Commit message: feat: new urdf for training

File: assets/URDF/big_bertha/Spyder_mg995_description.urdf (robot description, URDF)
Before this commit: robot SpdrBot, 17 links, 16 joints
Links:
- added link world
Joints:
- added joint world_to_base: type fixed, parent world, child base_link, origin xyz=0 0 0 rpy=1.5708 0 0

Commit message: feat: add inertial tags to fix null prim in usd spawn

File: assets/URDF/big_bertha/Spyder_mg995_description.urdf (robot description, URDF)
Before this commit: robot SpdrBot, 18 links, 17 joints
Links:
- removed link world
- link arm_a_1_1: geometry collision mesh filename=./meshes/arm_a_right.stl scale=0.001 0.001 0.001; collision mesh filename=./meshes/servo_mg995.stl scale=0.001 0.001 0.001
- link arm_a_2_1: geometry collision mesh filename=./meshes/arm_a_left.stl scale=0.001 0.001 0.001; collision mesh filename=./meshes/servo_mg995.stl scale=0.001 0.001 0.001
- link arm_a_3_1: geometry collision mesh filename=./meshes/arm_a_left.stl scale=0.001 0.001 0.001; collision mesh filename=./meshes/servo_mg995.stl scale=0.001 0.001 0.001
- link arm_a_4_1: geometry collision mesh filename=./meshes/arm_a_right.stl scale=0.001 0.001 0.001; collision mesh filename=./meshes/servo_mg995.stl scale=0.001 0.001 0.001
- link arm_b_1_1: geometry collision mesh filename=./meshes/arm_b.stl scale=0.001 0.001 0.001; visual mesh filename=./meshes/arm_b.stl scale=0.001 0.001 0.001
- link arm_b_2_1: geometry collision mesh filename=./meshes/arm_b.stl scale=0.001 0.001 0.001; visual mesh filename=./meshes/arm_b.stl scale=0.001 0.001 0.001
- link arm_b_3_1: geometry collision mesh filename=./meshes/arm_b.stl scale=0.001 0.001 0.001; visual mesh filename=./meshes/arm_b.stl scale=0.001 0.001 0.001
- link arm_b_4_1: geometry collision mesh filename=./meshes/arm_b.stl scale=0.001 0.001 0.001; visual mesh filename=./meshes/arm_b.stl scale=0.001 0.001 0.001
- link arm_c_1_1: geometry collision mesh filename=./meshes/arm_c_right.stl scale=0.001 0.001 0.001; collision mesh filename=./meshes/servo_mg995.stl scale=0.001 0.001 0.001
- link arm_c_2_1: geometry collision mesh filename=./meshes/arm_c_left.stl scale=0.001 0.001 0.001; collision mesh filename=./meshes/servo_mg995.stl scale=0.001 0.001 0.001
- link arm_c_3_1: geometry collision mesh filename=./meshes/arm_c_left.stl scale=0.001 0.001 0.001; collision mesh filename=./meshes/servo_mg995.stl scale=0.001 0.001 0.001
- link arm_c_4_1: geometry collision mesh filename=./meshes/arm_c_right.stl scale=0.001 0.001 0.001; collision mesh filename=./meshes/servo_mg995.stl scale=0.001 0.001 0.001
- link base_link: geometry collision mesh filename=./meshes/arm_perforated_plate_bottom.stl scale=0.001 0.001 0.001; collision mesh filename=./meshes/arm_perforated_plate_bottom.stl scale=0.001 0.001 0.001
- link circuit_box_link: mass 0.139015 -> 0.138015; geometry collision box size=0.102 0.1333 0.001; collision mesh filename=./meshes/body_standoffs.stl scale=0.001 0.001 0.001
- link ydlidar_link: mass 0.126000 -> 0.150000
Joints:
- removed joint world_to_base
- joint Revolute_110: limit lower=-1.57 upper=1.57 effort=1.18 velocity=5.5 -> lower=-1.57 upper=1.57; origin xyz=0.129 0.02 -0.015 rpy=0 -0.785 0 -> xyz=0.129 0.015 0.04 rpy=1.570796 -0 -0.785
- joint Revolute_111: limit lower=-1.57 upper=0.96 effort=1.18 velocity=5.5 -> lower=-1.57 upper=0.96
- joint Revolute_112: limit lower=0 upper=2.355 effort=1.18 velocity=5.5 -> lower=0 upper=2.355
- joint Revolute_113: limit lower=-1.57 upper=1.57 effort=1.18 velocity=5.5 -> lower=-1.57 upper=1.57; origin xyz=-0.015 0.02 0.002 rpy=0 0.785 0 -> xyz=-0.015 -0.002 0.04 rpy=1.570796 -0 0.785
- joint Revolute_114: limit lower=-1.57 upper=0.96 effort=1.18 velocity=5.5 -> lower=-1.57 upper=0.96
- joint Revolute_115: limit lower=0 upper=2.355 effort=1.18 velocity=5.5 -> lower=0 upper=2.355
- joint Revolute_116: limit lower=-1.57 upper=1.57 effort=1.18 velocity=5.5 -> lower=-1.57 upper=1.57; origin xyz=0.0027 0.02 0.145 rpy=0 2.355 0 -> xyz=0.0027 -0.145 0.04 rpy=1.570796 -0 2.355
- joint Revolute_117: limit lower=-1.57 upper=0.96 effort=1.18 velocity=5.5 -> lower=-1.57 upper=0.96
- joint Revolute_118: limit lower=0 upper=2.355 effort=1.18 velocity=5.5 -> lower=0 upper=2.355
- joint Revolute_119: limit lower=-1.57 upper=1.57 effort=1.18 velocity=5.5 -> lower=-1.57 upper=1.57; origin xyz=0.145 0.02 0.128 rpy=0 -2.355 0 -> xyz=0.145 -0.128 0.04 rpy=1.570796 -0 -2.355
- joint Revolute_120: limit lower=-1.57 upper=0.96 effort=1.18 velocity=5.5 -> lower=-1.57 upper=0.96
- joint Revolute_121: limit lower=0 upper=2.355 effort=1.18 velocity=5.5 -> lower=0 upper=2.355
- joint battery_joint: origin xyz=0.0657 0.0385 0.0657 rpy=1.57 0 0 -> xyz=0.0657 -0.0657 0.0585 rpy=3.140796 -0 0

Commit message: fix: cap calf flexion limit 2.355 to 2.0 rad to curb over-fold

File: assets/URDF/big_bertha/Spyder_mg995_description.urdf (robot description, URDF)
Before this commit: robot SpdrBot, 17 links, 16 joints
Joints:
- joint Revolute_112: limit lower=0 upper=2.355 -> lower=0 upper=2.0
- joint Revolute_115: limit lower=0 upper=2.355 -> lower=0 upper=2.0
- joint Revolute_118: limit lower=0 upper=2.355 -> lower=0 upper=2.0
- joint Revolute_121: limit lower=0 upper=2.355 -> lower=0 upper=2.0

Commit message: Revert "fix: cap calf flexion limit 2.355 to 2.0 rad to curb over-fold"
This reverts commit 5ad026145bf5b0985837c1c2b831e6855bd36655.

File: assets/URDF/big_bertha/Spyder_mg995_description.urdf (robot description, URDF)
Before this commit: robot SpdrBot, 17 links, 16 joints
Joints:
- joint Revolute_112: limit lower=0 upper=2.0 -> lower=0 upper=2.355
- joint Revolute_115: limit lower=0 upper=2.0 -> lower=0 upper=2.355
- joint Revolute_118: limit lower=0 upper=2.0 -> lower=0 upper=2.355
- joint Revolute_121: limit lower=0 upper=2.0 -> lower=0 upper=2.355
