Commit message: fix: move base_link to the body centre, repair stale IMU mesh path
What:
- Shift everything expressed in the base_link frame by -C, where C is
  base_link's inertial origin (0.06489606, -0.06499993): the four leg joint
  origins, battery_joint, and base_link's own inertial/visual/collision
  origins. x and y only.
- Repoint the IMU mesh at ./meshes/MPU_9265.stl.

Why:
- base_link sat 92 mm off the body centre and only 15 mm from leg 1's hip, so
  yaw commands pivoted the robot about one of its own legs rather than about
  itself. The policy tracks yaw at base_link, so this frame decides where it
  turns.
- After the shift the hip centroid is 0.53 mm from the origin (was 92 mm),
  all four hips sit at 101-103 mm radius, and base_link's inertial origin
  lands exactly on (0, 0).
- No geometry moves: child links keep their own frames, so the assembled
  robot is unchanged in world space. Only the frame moves.
- The URDF referenced ./meshes/mpu6050.stl, but that file was renamed to
  MPU_9265.stl. The converter resolved nothing and silently dropped the mesh
  from BOTH visual and collision, taking big_bertha_base.usd from 29.6 MB to
  25.5 MB. Left unfixed, v2.0.0 would have trained against different
  collision geometry than v1.2.0 for reasons unrelated to this change.

How:
- Applied by script, not by hand. 44 changed lines: 42 origins and the 2 mesh
  paths. No mass, inertia, limit or link name touched.
- USD regenerated; base.usd is within 141 bytes of the pre-move build, which
  is the origin text-length delta.

File: assets/URDF/big_bertha/Spyder_mg995_description.urdf (robot description, URDF)
Before this commit: robot SpdrBot, 17 links, 16 joints
Links:
- link circuit_box_link: geometry collision box size=0.102 0.1333 0.001; collision mesh filename=./meshes/MPU_9265.stl scale=0.001 0.001 0.001
Joints:
- joint Revolute_110: origin xyz=0.129 0.015 0.04 rpy=1.570796 -0 -0.785 -> xyz=0.06410394 0.07999993 0.04 rpy=1.570796 -0 -0.785
- joint Revolute_113: origin xyz=-0.015 -0.002 0.04 rpy=1.570796 -0 0.785 -> xyz=-0.07989606 0.06299993 0.04 rpy=1.570796 -0 0.785
- joint Revolute_116: origin xyz=0.0027 -0.145 0.04 rpy=1.570796 -0 2.355 -> xyz=-0.06219606 -0.08000007 0.04 rpy=1.570796 -0 2.355
- joint Revolute_119: origin xyz=0.145 -0.128 0.04 rpy=1.570796 -0 -2.355 -> xyz=0.08010394 -0.06300007 0.04 rpy=1.570796 -0 -2.355
- joint battery_joint: origin xyz=0.0657 -0.0657 0.0585 rpy=3.140796 -0 0 -> xyz=0.00080394 -0.00070007 0.0585 rpy=3.140796 -0 0
