Commit message: feat: urdf finalized with stl point cont and mpu9265

File: assets/URDF/big_bertha/Spyder_mg995_description_v2.urdf (robot description, URDF)
Before this commit: robot SpdrBot, 17 links, 16 joints
Links:
- link arm_c_1_1: mass 0.063683 -> 0.063687
- link arm_c_2_1: mass 0.063683 -> 0.063687
- link arm_c_3_1: mass 0.063683 -> 0.063687
- link arm_c_4_1: mass 0.063683 -> 0.063687
- link circuit_box_link: geometry collision box size=0.102 0.1333 0.001; collision mesh filename=./meshes/MPU_9250.stl scale=0.001 0.001 0.001

Commit message: fix: mpu rename

File: assets/URDF/big_bertha/Spyder_mg995_description_v2.urdf (robot description, URDF)
Before this commit: robot SpdrBot, 17 links, 16 joints
Links:
- link circuit_box_link: geometry collision box size=0.102 0.1333 0.001; collision mesh filename=./meshes/MPU_9265.stl scale=0.001 0.001 0.001
